Commit message: change lidar rotate config in mirs.urdf

File: src/mirs_mg5/mirs/urdf/mirs.urdf (robot description, URDF)
Before this commit: robot cleaning_robot, 6 links, 5 joints
Joints:
- joint lidar_joint: origin xyz=0 0 0.105 rpy=3.14159 0 0 -> xyz=0 0 0.105 rpy=0 0 0

Commit message: fix: AMCLの運動モデルパラメータを調整

File: src/mirs_mg5/mirs/urdf/mirs.urdf (robot description, URDF)
Before this commit: robot cleaning_robot, 6 links, 5 joints
Joints:
- joint base_joint: child base_link -> base_footprint; origin xyz=0 0 0.0391 rpy=0 0 0 -> xyz=0 0 -0.0391 rpy=0 0 0; parent base_footprint -> base_link
- joint left_wheel_joint: origin xyz=0 0.212 0 rpy=0 0 0 -> xyz=0 0.19 0 rpy=0 0 0
- joint right_wheel_joint: origin xyz=0 -0.212 0 rpy=0 0 0 -> xyz=0 -0.19 0 rpy=0 0 0

Commit message: feat: ナビゲーションパラメータを調整し、マップ設定を更新し、joint_state_publisherを追加

File: src/mirs_mg5/mirs/urdf/mirs.urdf (robot description, URDF)
Before this commit: robot cleaning_robot, 6 links, 5 joints
Joints:
- joint left_wheel_joint: origin xyz=0 0.19 0 rpy=0 0 0 -> xyz=0 0.195 0 rpy=0 0 0
- joint right_wheel_joint: origin xyz=0 -0.19 0 rpy=0 0 0 -> xyz=0 -0.195 0 rpy=0 0 0
